File: hardware/stnstarter.kicad_pcb (KiCad board)
At the start: 2 copper layers, 52.6 x 60 mm, 52 parts, among them J1 AAF1202FNF, J2 WD-X16161, J3 Conn_01x02, SW1 SW_Push, SW2 SW_Push, SW3 SW_Push, U1 AP3015, U2 Pico, U3 NC7WZ16P6X, U4 CAT4139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

Commit message: Rev 0.2
Parts:
- removed C12, C13, C14: 4.7uF, Capacitor_SMD:C_0603_1608Metric
- removed J2: WD-X16161, footprints:FPC_20
- removed J3: Conn_01x02, Connector_PinHeader_2.54mm:PinHeader_1x02_P2.54mm_Vertical
- removed R10, R11, R13, R14: 10K, Resistor_SMD:R_0402_1005Metric
- removed R12: 75K, Resistor_SMD:R_0402_1005Metric
- removed R15, R16, R17, R18: 10, Resistor_SMD:R_0402_1005Metric
- removed U5: LM324, Package_SO:TSSOP-14_4.4x5mm_P0.65mm
- added L3: 10uH, footprints:L_1212, F.Cu at (105.3, 79.1)
- C11: value 4.7uF -> 100nF; footprint Capacitor_SMD:C_0603_1608Metric -> Capacitor_SMD:C_0402_1005Metric
- C4: value 100nF -> 220nF
- J1: value AAF1202FNF -> Conn_01x14; footprint Connector_FFC-FPC:TE_1-84952-2_1x12-1MP_P1.0mm_Horizontal -> Connector_PinSocket_2.00mm:PinSocket_1x13_P2.00mm_Vertical
- U1: value AP3015 -> 74HC245; footprint Package_TO_SOT_SMD:TSOT-23-5 -> Package_DFN_QFN:WQFN-20-1EP_2.5x4.5mm_P0.5mm_EP1x2.9mm
- U3: value NC7WZ16P6X -> LT1617; footprint Package_TO_SOT_SMD:SOT-363_SC-70-6 -> Package_TO_SOT_SMD:SOT-23-5
- moved U1 40.9 mm to (121.2, 111.0), turned to -90 degrees
- moved C9 17.7 mm to (136.0, 111.7)
- moved R9 17.6 mm to (136.0, 114.5)
- moved D2 13.8 mm to (138.5, 112.6), turned to -90 degrees
- moved C4 12.5 mm to (104.2, 73.8)
- moved U3 10.2 mm to (109.3, 71.9), turned to 90 degrees
- moved C5 9.21 mm to (141.9, 109.2), turned to 0 degrees
- moved L2 8.12 mm to (142.0, 112.7), turned to -90 degrees
- moved J1 6.04 mm to (107.7, 114.5), turned to 90 degrees
- moved C6 4.91 mm to (145.4, 109.7), turned to 180 degrees
- moved R3 3.64 mm to (147.6, 109.7), turned to 180 degrees
- moved U4 2.52 mm to (146.0, 112.7), turned to 90 degrees
- moved U2 2.40 mm to (127.1, 95.4)
- moved R8 2.37 mm to (148.6, 113.7), turned to 90 degrees
- moved C2 2.22 mm to (109.7, 78.2)
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Connections:
- C11 pad 2: /LCD_V1 -> +5V
- C2 pad 2: VPP -> VEE
- C3 pad 2: VPP -> VEE
- C4 pad 1: GND -> Net-(L1-Pad2)
- C4 pad 2: +3V3 -> Net-(D1-Pad2)
- D1 pad 1: VPP -> GND
- J1 pad 1: /D3 -> unconnected-(J1-Pad1)
- J1 pad 10: /VCLK -> /HSYNCS
- J1 pad 11: /VSYNC -> /VSYNCS
- J1 pad 12: /LCD_EN -> /LEDK
- J1 pad 2: /D2 -> VEE
- J1 pad 3: /D1 -> /D0S
- J1 pad 4: /D0 -> /D1S
- J1 pad 5: VPP -> /D2S
- J1 pad 6: GND -> /D3S
- J1 pad 7: +3V3 -> GND
- J1 pad 8: /AC -> +5V
- J1 pad 9: /HSYNC -> /VCLKS
- L1 pad 2: Net-(D1-Pad2) -> Net-(L1-Pad2)
- R3 pad 1: /LCD_EN -> /BL_EN
- R4 pad 2: VPP -> VEE
- U1 pad 1: Net-(D1-Pad2) -> +5V
- U1 pad 2: GND -> /VSYNC
- U1 pad 3: Net-(R4-Pad1) -> /HSYNC
- U1 pad 4: /LCD_EN -> /VCLK
- U2 pad 10: /LCD_EN -> /D3
- U2 pad 11: /D0 -> /VCLK
- U2 pad 12: /D1 -> /HSYNC
- U2 pad 14: /D2 -> /VSYNC
- U2 pad 15: /D3 -> unconnected-(U2-Pad15)
- U2 pad 16: /D4 -> unconnected-(U2-Pad16)
- U2 pad 17: /D5 -> unconnected-(U2-Pad17)
- U2 pad 19: /D6 -> /BL_EN
- U2 pad 20: /D7 -> unconnected-(U2-Pad20)
- U2 pad 32: /PWM1 -> /LCD_EN
- U2 pad 6: /HSYNC -> /D0
- U2 pad 7: /VCLK -> /D1
- U2 pad 9: /VSYNC -> /D2
- U3 pad 1: /PWM0 -> Net-(L1-Pad2)
- U3 pad 3: /PWM1 -> Net-(R4-Pad1)
- U3 pad 4: Net-(J3-Pad2) -> /LCD_EN
- U3 pad 5: +3V3 -> +5V
- U4 pad 4: /LCD_EN -> /BL_EN
Routing:
- net VPP: track 92.1 -> 0.00 mm, vias 2 -> 0
- net /LCD_EN: track 106.1 -> 31.1 mm, vias 3 -> 0
- net +3V3: track 136.6 -> 72.2 mm, vias 8 -> 4
- net /D1: track 56.6 -> 6.14 mm, vias 2 -> 0
- net /D2: track 56.3 -> 7.63 mm, vias 2 -> 0
- net /D3: track 58.2 -> 9.76 mm, vias 2 -> 0
- net /D0: track 55.5 -> 8.10 mm, vias 2 -> 0
- net /AC: track 40.5 -> 0.00 mm
- net VEE: track 0.00 -> 38.6 mm, vias 0 -> 1
- net +5V: track 93.5 -> 118.9 mm, vias 1 -> 5
- net /HSYNC: track 35.8 -> 12.9 mm
- net /VCLK: track 32.9 -> 10.8 mm
- net /D7: track 21.9 -> 0.00 mm, vias 1 -> 0
- net /D4: track 21.3 -> 0.00 mm, vias 1 -> 0
- net /D6: track 21.0 -> 0.00 mm, vias 1 -> 0
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- added copper zone on F.Cu, net +5V
- added copper zone on F.Cu, net /LEDA
- added copper zone on F.Cu, net Net-(D2-Pad2)
- added copper zone on F.Cu, net Net-(L1-Pad2)
- added copper zone on F.Cu, net VEE
Other:
- board size 52.6 x 60 mm -> 52.6 x 50.6 mm
- board text removed: "Wenting 2022 R0.1"
