File: hardware/stnstarter.kicad_sch (KiCad schematic)
At the start: 52 parts, among them J1 AAF1202FNF, J2 WD-X16161, J3 Conn_01x02, SW1 SW_Push, SW2 SW_Push, SW3 SW_Push, U1 AP3015, U2 Pico, U3 NC7WZ16P6X, U4 CAT4139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

Commit message: Rev 0.2
Parts:
- removed C12, C13, C14: 4.7uF, Capacitor_SMD:C_0603_1608Metric, symbol Device:C
- removed J1: AAF1202FNF, Connector_FFC-FPC:TE_1-84952-2_1x12-1MP_P1.0mm_Horizontal, symbol Connector_Generic:Conn_01x12
- removed J2: WD-X16161, footprints:FPC_20, symbol Connector_Generic:Conn_01x20
- removed J3: Conn_01x02, Connector_PinHeader_2.54mm:PinHeader_1x02_P2.54mm_Vertical, symbol Connector_Generic:Conn_01x02
- removed R10, R11, R13, R14: 10K, Resistor_SMD:R_0402_1005Metric, symbol Device:R
- removed R12: 75K, Resistor_SMD:R_0402_1005Metric, symbol Device:R
- removed R15, R16, R17, R18: 10, Resistor_SMD:R_0402_1005Metric, symbol Device:R
- removed U1: AP3015, Package_TO_SOT_SMD:TSOT-23-5, symbol symbols:SY7152
- removed U3: NC7WZ16P6X, Package_TO_SOT_SMD:SOT-363_SC-70-6, symbol RPi_Pico:NC7WZ16P6X
- removed U5: LM324, Package_SO:SOIC-16_3.9x9.9mm_P1.27mm, symbol Amplifier_Operational:LM324
- added J1: Conn_01x14, Connector_PinSocket_2.00mm:PinSocket_1x13_P2.00mm_Vertical, symbol Connector_Generic:Conn_01x14
- added L3: 10uH, footprints:L_1212, symbol Device:L
- added U1: 74HC245, Package_DFN_QFN:WQFN-20-1EP_2.5x4.5mm_P0.5mm_EP1x2.9mm, symbol 74xx:74HC245
- added U3: LT1617, Package_TO_SOT_SMD:SOT-23-5, symbol symbols:LT1617
- C11: value 4.7uF -> 100nF; footprint Capacitor_SMD:C_0603_1608Metric -> Capacitor_SMD:C_0402_1005Metric
- C4: value 100nF -> 220nF
Connections:
- net LCD_V1 is gone; now on net +5V: C11.2
- net PWM1 is gone; now on net LCD_EN: U2.32 (GPIO27_ADC1)
- net +3V3: no longer C4.2
- net +5V: now also J1.8 (Pin_8), U1.1 (A->B), U1.20 (VCC), U1.5 (A3), U3.5 (VIN)
- net D0: now also U2.6 (GPIO4), U1.9 (A7); no longer U2.11 (GPIO8)
- net D1: now also U2.7 (GPIO5), U1.8 (A6); no longer U2.12 (GPIO9)
- net D2: now also U2.9 (GPIO6), U1.7 (A5); no longer U2.14 (GPIO10)
- net D3: now also U2.10 (GPIO7), U1.6 (A4); no longer U2.15 (GPIO11)
- net GND: now also D1.1 (K), J1.7 (Pin_7), U1.10 (GND), U1.19 (CE), U3.2 (GND); no longer C4.1
- net HSYNC: now also U2.12 (GPIO9), U1.3 (A1); no longer U2.6 (GPIO4)
- net LCD_EN: now also U3.4 (RUN); no longer R3.1, U2.10 (GPIO7), U4.4 (~{SHDN})
- net LEDA: now also J1.13 (Pin_13)
- net LEDK: now also J1.12 (Pin_12)
- net VCLK: now also U2.11 (GPIO8), U1.4 (A2); no longer U2.7 (GPIO5)
- net VSYNC: now also U2.14 (GPIO10), U1.2 (A0); no longer U2.9 (GPIO6)
- net at L1.2: now also C4.1, U3.1 (LX); no longer D1.2 (A)
- net at R4.1, RV1.1: now also U3.3 (NFB)
- net D4: no longer names the net of U2.16 (GPIO12)
- net D5: no longer names the net of U2.17 (GPIO13)
- net D6 renamed BL_EN
- net BL_EN: now also R3.1, U4.4 (~{SHDN})
- net D7: no longer names the net of U2.20 (GPIO15)
- net VPP renamed VEE
- net VEE: now also J1.2 (Pin_2), L3.2; no longer D1.1 (K)
- new net: C4.2, D1.2 (A), L3.1
- new net D0S: J1.3 (Pin_3), U1.11 (B7)
- new net D1S: J1.4 (Pin_4), U1.12 (B6)
- new net D2S: J1.5 (Pin_5), U1.13 (B5)
- new net D3S: J1.6 (Pin_6), U1.14 (B4)
- new net HSYNCS: J1.10 (Pin_10), U1.17 (B1)
- new net VCLKS: J1.9 (Pin_9), U1.16 (B2)
- new net VSYNCS: J1.11 (Pin_11), U1.18 (B0)
- no-connect marks 3 -> 5
Other:
- moved on the sheet: C1, C2, C3, C5, C6, C8, C9, D1, D2, L1, L2, R3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
